File: tgam_breakout/tgam_breakout.brd (EAGLE design)
At the start: 33 x 43.2 mm, 14 parts, among them X1 332-06, X2 332-10

Commit message: seems some inconsistencies were left over
Parts:
- removed JP1: (no value), pinhead:1X04
Connections:
- removed net RDX: JP1.4
- net GND: no longer JP1.3
- net TXD: no longer JP1.2
- net VCC: no longer JP1.1
Routing:
- net VCC: track 16.7 -> 0.00 mm
- net RXD: track 10.8 -> 0.00 mm
- net TXD: track 8.61 -> 0.00 mm
- net REF: track 7.03 -> 0.00 mm
Changed lines of the file:
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@@
 <element name="GND_ELEL" library="SparkFun-Connectors" package="U.FL" value="U.FL" x="6.35" y="31.75"/>
 <element name="REF_EL" library="SparkFun-Connectors" package="U.FL" value="U.FL" x="6.35" y="6.35"/>
-<element name="JP1" library="pinhead" package="1X04" value="" x="26.67" y="2.54" smashed="yes">
-<attribute name="VALUE" x="21.59" y="-0.635" size="1.27" layer="27"/>
-</element>
 <element name="PAD1" library="wirepad" package="SMD2,54-5,08" value="" x="6.35" y="19.05" smashed="yes" rot="MR0">
 <attribute name="VALUE" x="6.35" y="19.05" size="0.0254" layer="28" rot="MR0"/>
@@
 <wire x1="27.178" y1="32.893" x2="27.0698" y2="33.0106" width="0.1524" layer="1"/>
 <wire x1="28.194" y1="32.512" x2="28.06294375" y2="32.402" width="0.1524" layer="1"/>
+<wire x1="27.835" y1="38.735" x2="30.585" y2="38.735" width="0" layer="19" extent="1-1"/>
+<wire x1="27.0698" y1="33.0106" x2="27.835" y2="38.735" width="0" layer="19" extent="1-1"/>
 </signal>
 <signal name="GND_EL">
@@
 <vertex x="20.955" y="36.195"/>
 </polygon>
+<wire x1="16.405" y1="38.735" x2="19.155" y2="38.735" width="0" layer="19" extent="1-1"/>
+<wire x1="21.0698" y1="33.0106" x2="19.155" y2="38.735" width="0" layer="19" extent="1-1"/>
 </signal>
 <signal name="REF">
 <contactref element="REF" pad="P$3"/>
 <contactref element="X2" pad="3"/>
-<wire x1="17.78" y1="37.21" x2="20.065" y2="34.925" width="0.4064" layer="1" curve="90"/>
-<wire x1="20.065" y1="34.925" x2="20.32" y2="34.925" width="0.4064" layer="1"/>
-<wire x1="20.32" y1="34.925" x2="21.1554" y2="34.925" width="0.4064" layer="1"/>
-<wire x1="21.1554" y1="34.925" x2="23.0698" y2="33.0106" width="0.4064" layer="1" curve="-90"/>
+<wire x1="23.0698" y1="33.0106" x2="17.78" y2="37.21" width="0" layer="19" extent="1-1"/>
 </signal>
 <signal name="VCC">
@@
 <contactref element="C1" pad="1"/>
 <contactref element="C2" pad="1"/>
-<wire x1="19.685" y1="3.429" x2="17.526" y2="3.429" width="0.1524" layer="1"/>
-<wire x1="17.526" y1="3.429" x2="16.51" y2="3.429" width="0.1524" layer="1"/>
-<wire x1="16.51" y1="3.429" x2="16.51" y2="3.49" width="0.1524" layer="1"/>
-<wire x1="19.685" y1="3.429" x2="19.685" y2="3.49" width="0.1524" layer="1"/>
-<wire x1="17.526" y1="7.747" x2="17.526" y2="3.429" width="0.1524" layer="1"/>
-<wire x1="17.526" y1="7.747" x2="17.415" y2="7.779" width="0.1524" layer="1"/>
-<wire x1="18.415" y1="10.795" x2="19.304" y2="11.684" width="0.1524" layer="16"/>
-<wire x1="18.415" y1="8.763" x2="18.415" y2="10.795" width="0.1524" layer="16"/>
-<wire x1="17.526" y1="7.874" x2="18.415" y2="8.763" width="0.1524" layer="16"/>
-<wire x1="19.304" y1="11.684" x2="19.415" y2="11.779" width="0.1524" layer="16"/>
-<wire x1="17.526" y1="7.874" x2="17.415" y2="7.779" width="0.1524" layer="16"/>
-<contactref element="JP1" pad="1"/>
-<wire x1="19.685" y1="2.54" x2="22.86" y2="2.54" width="0.1524" layer="1"/>
-<wire x1="19.685" y1="3.429" x2="19.685" y2="2.54" width="0.1524" layer="1"/>
-<wire x1="19.685" y1="3.429" x2="19.685" y2="3.49" width="0.1524" layer="1"/>
+<wire x1="17.415" y1="7.779" x2="19.415" y2="11.779" width="0" layer="19" extent="1-1"/>
+<wire x1="16.51" y1="3.49" x2="17.415" y2="7.779" width="0" layer="19" extent="1-1"/>
+<wire x1="19.685" y1="3.49" x2="16.51" y2="3.49" width="0" layer="19" extent="1-1"/>
 </signal>
 <signal name="RXD">
 <contactref element="X1" pad="4"/>
-<wire x1="24.892" y1="4.318" x2="19.431" y2="9.779" width="0.1524" layer="16"/>
-<wire x1="27.94" y1="4.318" x2="24.892" y2="4.318" width="0.1524" layer="16"/>
-<wire x1="19.431" y1="9.779" x2="19.415" y2="9.779" width="0.1524" layer="16"/>
 </signal>
 <signal name="TXD">
 <contactref element="X1" pad="6"/>
-<contactref element="JP1" pad="2"/>
-<wire x1="20.955" y1="7.747" x2="19.431" y2="7.747" width="0.1524" layer="16"/>
-<wire x1="25.4" y1="3.302" x2="20.955" y2="7.747" width="0.1524" layer="16"/>
-<wire x1="25.4" y1="2.54" x2="25.4" y2="3.302" width="0.1524" layer="16"/>
-<wire x1="19.431" y1="7.747" x2="19.415" y2="7.779" width="0.1524" layer="16"/>
 </signal>
 <signal name="GND">
@@
 <vertex x="36.195" y="-1.27"/>
 </polygon>
-<contactref element="JP1" pad="3"/>
+<wire x1="17.415" y1="9.779" x2="17.415" y2="11.779" width="0" layer="19" extent="1-1"/>
+<wire x1="16.51" y1="1.59" x2="17.415" y2="9.779" width="0" layer="19" extent="1-1"/>
+<wire x1="19.685" y1="1.59" x2="16.51" y2="1.59" width="0" layer="19" extent="1-1"/>
 </signal>
 <signal name="EEG2">
@@
 <wire x1="6.35" y1="7.62" x2="6.35" y2="7.725" width="0.1524" layer="1"/>
 </signal>
-<signal name="RDX">
-<contactref element="JP1" pad="4"/>
-</signal>
 </signals>

Commit message: Oh fsck! I had switched reference electrode and shield connections...
Parts:
- added JP1: (no value), pinhead:1X04
Connections:
- net GND: now also GND_EL.P$1, GND_EL.P$2, JP1.3
- net REF: now also X2.1; no longer X2.3
- net REF_SHD: now also X2.3; no longer X2.1
- net RXD: now also JP1.4
- net TXD: now also JP1.2
- net VCC: now also JP1.1
Routing:
- net REF: track 0.00 -> 5.56 mm
- net EEG_SHD: track 1.61 -> 3.81 mm
Changed lines of the file:
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@@
 <attribute name="VALUE" x="6.35" y="6.35" size="0.0254" layer="28" rot="MR0"/>
+</element>
+<element name="JP1" library="pinhead" package="1X04" value="" x="26.67" y="2.54" smashed="yes">
+<attribute name="VALUE" x="21.59" y="-0.635" size="1.27" layer="27"/>
 </element>
 </elements>
@@
 <vertex x="31.115" y="30.48"/>
 </polygon>
-<wire x1="27.559" y1="32.512" x2="27.178" y2="32.893" width="0.1524" layer="1"/>
-<wire x1="27.813" y1="32.512" x2="27.559" y2="32.512" width="0.1524" layer="1"/>
-<wire x1="27.94" y1="32.639" x2="27.813" y2="32.512" width="0.1524" layer="1"/>
-<wire x1="28.067" y1="32.639" x2="27.94" y2="32.639" width="0.1524" layer="1"/>
-<wire x1="28.194" y1="32.512" x2="28.067" y2="32.639" width="0.1524" layer="1"/>
-<wire x1="27.178" y1="32.893" x2="27.0698" y2="33.0106" width="0.1524" layer="1"/>
-<wire x1="28.194" y1="32.512" x2="28.06294375" y2="32.402" width="0.1524" layer="1"/>
-<wire x1="27.835" y1="38.735" x2="30.585" y2="38.735" width="0" layer="19" extent="1-1"/>
-<wire x1="27.0698" y1="33.0106" x2="27.835" y2="38.735" width="0" layer="19" extent="1-1"/>
+<wire x1="27.305" y1="33.02" x2="27.305" y2="34.29" width="0.4064" layer="1"/>
+<wire x1="27.305" y1="34.29" x2="27.305" y2="31.75" width="0.4064" layer="1"/>
 </signal>
 <signal name="GND_EL">
@@
 <contactref element="REF" pad="P$1"/>
 <contactref element="REF" pad="P$2"/>
-<contactref element="X2" pad="1"/>
 <polygon width="0.4064" layer="1" isolate="0.254">
 <vertex x="20.955" y="40.64"/>
@@
 <vertex x="14.605" y="30.48"/>
 <vertex x="23.495" y="30.48"/>
-<vertex x="23.495" y="35.56"/>
-<vertex x="20.955" y="36.195"/>
+<vertex x="23.495" y="34.925"/>
+<vertex x="20.955" y="35.56"/>
 </polygon>
-<wire x1="16.405" y1="38.735" x2="19.155" y2="38.735" width="0" layer="19" extent="1-1"/>
-<wire x1="21.0698" y1="33.0106" x2="19.155" y2="38.735" width="0" layer="19" extent="1-1"/>
+<contactref element="X2" pad="3"/>
 </signal>
 <signal name="REF">
 <contactref element="REF" pad="P$3"/>
-<contactref element="X2" pad="3"/>
-<wire x1="23.0698" y1="33.0106" x2="17.78" y2="37.21" width="0" layer="19" extent="1-1"/>
+<contactref element="X2" pad="1"/>
+<wire x1="17.78" y1="37.21" x2="17.78" y2="36.3004" width="0.4064" layer="1"/>
+<wire x1="17.78" y1="36.3004" x2="21.0698" y2="33.0106" width="0.4064" layer="1" curve="90"/>
 </signal>
 <signal name="VCC">
@@
 <contactref element="C1" pad="1"/>
 <contactref element="C2" pad="1"/>
+<contactref element="JP1" pad="1"/>
 <wire x1="17.415" y1="7.779" x2="19.415" y2="11.779" width="0" layer="19" extent="1-1"/>
 <wire x1="16.51" y1="3.49" x2="17.415" y2="7.779" width="0" layer="19" extent="1-1"/>
 <wire x1="19.685" y1="3.49" x2="16.51" y2="3.49" width="0" layer="19" extent="1-1"/>
+<wire x1="22.86" y1="2.54" x2="19.685" y2="3.49" width="0" layer="19" extent="1-1"/>
 </signal>
 <signal name="RXD">
 <contactref element="X1" pad="4"/>
+<contactref element="JP1" pad="4"/>
+<wire x1="19.415" y1="9.779" x2="30.48" y2="2.54" width="0" layer="19" extent="1-1"/>
 </signal>
 <signal name="TXD">
 <contactref element="X1" pad="6"/>
+<contactref element="JP1" pad="2"/>
+<wire x1="19.415" y1="7.779" x2="25.4" y2="2.54" width="0" layer="19" extent="1-1"/>
 </signal>
 <signal name="GND">
@@
 <vertex x="36.195" y="-1.27"/>
 </polygon>
-<wire x1="17.415" y1="9.779" x2="17.415" y2="11.779" width="0" layer="19" extent="1-1"/>
-<wire x1="16.51" y1="1.59" x2="17.415" y2="9.779" width="0" layer="19" extent="1-1"/>
-<wire x1="19.685" y1="1.59" x2="16.51" y2="1.59" width="0" layer="19" extent="1-1"/>
+<contactref element="JP1" pad="3"/>
+<contactref element="GND_EL" pad="P$2"/>
+<contactref element="GND_EL" pad="P$1"/>
 </signal>
 <signal name="EEG2">
